Commit message: resourceupdate1

File: resources/grav.urdf (robot description, URDF)
Before this commit: robot flexiv_GN01, 14 links, 13 joints
Links:
- link base_link: geometry collision mesh filename=meshes/grav/collision/base.stl scale=0.001 0.001 0.001; visual mesh filename=meshes/grav/visual/base.stl scale=0.001 0.001 0.001
- link left_finger_mount: geometry visual mesh filename=meshes/grav/visual/finger_mount.stl scale=0.001 0.001 0.001
- link left_finger_tip: geometry collision mesh filename=meshes/grav/collision/finger_tip.stl scale=0.001 0.001 0.001; visual mesh filename=meshes/grav/visual/finger_tip.obj scale=0.001 0.001 0.001
- link left_inner_bar: geometry visual mesh filename=meshes/grav/visual/inner_bar.stl scale=0.001 0.001 0.001
- link left_outer_bar: geometry visual mesh filename=meshes/grav/visual/outer_bar.stl scale=0.001 0.001 0.001
- link right_finger_mount: geometry visual mesh filename=meshes/grav/visual/finger_mount.stl scale=0.001 0.001 0.001
- link right_finger_tip: geometry collision mesh filename=meshes/grav/collision/finger_tip.stl scale=0.001 0.001 0.001; visual mesh filename=meshes/grav/visual/finger_tip.obj scale=0.001 0.001 0.001
- link right_inner_bar: geometry visual mesh filename=meshes/grav/visual/inner_bar.stl scale=0.001 0.001 0.001
- link right_outer_bar: geometry visual mesh filename=meshes/grav/visual/outer_bar.stl scale=0.001 0.001 0.001
